File: LIFFY/KiCAD/LIFFY_KICAD/LIFFY_KICAD.kicad_pcb (KiCad board)
At the start: 2 copper layers, 72 x 150 mm, 89 parts, among them IC1 MC9S08MP16xLC, J1 VIN, J10 M1, J11 M2, J12 M3, J13 LEDBAR2, J14 VIN2, J15 Program_Pins, J16 CONN_I2C, J17 M4, J18 CON_REL1, J19 CON_REL2, J2 pH, J20 CON_REL3, J21 CONN_UART, J22 CON_REL4, J3 TDS, J4 LDR_CONECTOR, J5 DHT11, J6 LEVEL_SENSOR2, J7 LEDBAR1, J8 5V_OUT, J9 LEVEL_SENSOR1, K1 FINDER-36.11, K2 FINDER-36.11, K3 FINDER-36.11, K4 FINDER-36.11, Q1 IRF3205, Q2 IRF3205, SW1 SW_DIP_x04, U1 LM358, U2 LM358, U3 PC817, U4 MIC4427, U5 PC817, U6 ULN2003A, U7 AP63205WU, U8 ULN2003A, Y1 Crystal 4 MHz

Commit message: V2 PCB ADDED
Parts:
- removed C12, C13: 1n, Capacitor_SMD:C_0201_0603Metric
- removed RV4: Varistor_6V, Capacitor_SMD:C_0805_2012Metric
- added C18: 100n, Capacitor_SMD:C_0201_0603Metric, F.Cu at (111.3, 146.8)
- added C19: 100n, Capacitor_SMD:C_0201_0603Metric, F.Cu at (107.7, 120.4)
- added L2: 27n, Inductor_SMD:L_0805_2012Metric, F.Cu at (86.4, 81.3)
- J15, J16, J21: footprint Connector_PinHeader_1.00mm:PinHeader_1x04_P1.00mm_Vertical -> Connector_PinHeader_2.54mm:PinHeader_1x04_P2.54mm_Vertical
- moved U8 51.9 mm to (79.2, 90.4), turned to -90 degrees
- moved J21 43.5 mm to (84.3, 64.3), turned to 180 degrees
- moved J15 33.6 mm to (111.3, 76.7), turned to 180 degrees
- moved C9 32.2 mm to (86.0, 27.4), turned to 0 degrees
- moved R11 32.2 mm to (106.2, 114.6), turned to 90 degrees
- moved R23 32.0 mm to (80.3, 61.5)
- moved R24 30.4 mm to (80.1, 58.4)
- moved R19 30.1 mm to (114.8, 76.7)
- moved C8 28.0 mm to (85.9, 30.5)
- moved U4 27.0 mm to (84.3, 37.1), turned to -90 degrees
- moved R9 25.2 mm to (108.7, 147.1), turned to -90 degrees
- moved R21 24.8 mm to (115.0, 72.1)
- moved J16 24.0 mm to (93.2, 51.3)
- moved U5 23.4 mm to (110.2, 110.2), turned to 180 degrees
- moved R10 21.9 mm to (107.4, 129.5)
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Connections:
- net Net-(C15-Pad2) renamed /Fuente Conmutada 5V/SW
- C7 pad 2: +5V -> Net-(C7-Pad2)
- IC1 pad 21: +5V -> Net-(C7-Pad2)
Routing:
- net +12V: track 0.00 -> 242.3 mm, vias 0 -> 11
- net GND: track 0.00 -> 132.8 mm, vias 0 -> 33
- net /Sensores LIFFY/TEMP_HUM: track 0.00 -> 119.8 mm, vias 0 -> 2
- net +5V: track 0.00 -> 110.3 mm, vias 0 -> 31
- net /Sensores LIFFY/pH_DATA: track 0.00 -> 99.7 mm, vias 0 -> 4
- net /DIPSWITCHES/DIP3: track 0.00 -> 98.9 mm, vias 0 -> 3
- net /Sensores LIFFY/LDR_DATA: track 0.00 -> 84.0 mm, vias 0 -> 2
- net /Sensores LIFFY/TDS_DATA: track 0.00 -> 83.1 mm
- net Net-(K1-PadA2): track 0.00 -> 80.8 mm
- net /Sensores LIFFY/LV2: track 0.00 -> 62.4 mm, vias 0 -> 2
- net Net-(K2-PadA2): track 0.00 -> 60.3 mm
- net /DIPSWITCHES/DIP2: track 0.00 -> 56.2 mm, vias 0 -> 6
- net /Comunic. & Program./SDA_PIN: track 0.00 -> 55.5 mm
- net /Driver MOSFET para PWM 2 Outputs/PWM_A: track 0.00 -> 54.4 mm, vias 0 -> 2
- net /Sensores LIFFY/LV1: track 0.00 -> 51.5 mm, vias 0 -> 2
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- added copper zone on In2.Cu, net +12V
- added copper zone on F.Cu, net +5V
- added copper zone on In2.Cu, net +5V
- added copper zone on In1.Cu, net GND
Other:
- copper layers 2 -> 4
- board text removed: "PRUEBA"
