File: LIFFY/KiCAD/LIFFY_KICAD/LIFFY_KICAD.kicad_pcb (KiCad board)
At the start: 4 copper layers, 72 x 150 mm, 88 parts, among them IC1 MC9S08MP16xLC, J1 VIN, J10 M1, J11 M2, J12 M3, J13 LEDBAR2, J14 VIN2, J15 Program_Pins, J16 CONN_I2C, J17 M4, J18 CON_REL1, J19 CON_REL2, J2 pH, J20 CON_REL3, J21 CONN_UART, J22 CON_REL4, J3 TDS, J4 LDR_CONECTOR, J5 DHT11, J6 LEVEL_SENSOR2, J7 LEDBAR1, J8 5V_OUT, J9 LEVEL_SENSOR1, K1 FINDER-36.11, K2 FINDER-36.11, K3 FINDER-36.11, K4 FINDER-36.11, Q1 IRF3205, Q2 IRF3205, SW1 SW_DIP_x04, U1 LM358, U2 LM358, U3 PC817, U4 MIC4427, U5 PC817, U6 ULN2003A, U7 AP63205WU, U8 ULN2003A, Y1 Crystal 4 MHz

Commit message: V5 Aprobado
Routing:
- net /Motor Drivers/PW_MOTOR2: track 24.4 -> 30.7 mm
- net /Driver MOSFET para PWM 2 Outputs/PWM_A: track 54.9 -> 52.7 mm
- net +12V: track 228.5 -> 230.4 mm
Changed lines of the file:
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@@
   (gr_rect (start 55.88 22.86) (end 127.88 172.86) (layer "Edge.Cuts") (width 0.1) (fill none))
   (target plus (at 55.88 172.72) (size 5) (width 0.1) (layer "Edge.Cuts"))
-  (segment (start 82.212078 37.084) (end 80.772 37.084) (width 0.3048) (layer "F.Cu") (net 1))
   (segment (start 87.33 134.716) (end 78.328 134.716) (width 1.016) (layer "F.Cu") (net 1))
+  (segment (start 79.502 35.265919) (end 84.287919 30.48) (width 0.3048) (layer "F.Cu") (net 1))
   (segment (start 78.39 99.156) (end 82.392 99.156) (width 1.016) (layer "F.Cu") (net 1))
+  (segment (start 83.693 39.559001) (end 83.693 38.564922) (width 0.3048) (layer "F.Cu") (net 1))
   (segment (start 84.901989 30.48) (end 84.901989 28.513989) (width 0.3048) (layer "F.Cu") (net 1))
   (segment (start 110.357488 33.02) (end 110.357488 32.069989) (width 0.762) (layer "F.Cu") (net 1))
   (segment (start 59.436 91.948) (end 64.516 86.868) (width 1.016) (layer "F.Cu") (net 1))
   (segment (start 74.803 94.361) (end 74.803 92.899) (width 1.016) (layer "F.Cu") (net 1))
-  (segment (start 80.772 33.995919) (end 84.287919 30.48) (width 0.3048) (layer "F.Cu") (net 1))
   (segment (start 87.33 99.156) (end 82.392 99.156) (width 1.016) (layer "F.Cu") (net 1))
   (segment (start 113.284 32.004) (end 110.4235 32.004) (width 1.016) (layer "F.Cu") (net 1))
-  (segment (start 82.392 99.156) (end 82.296 99.06) (width 1.016) (layer "F.Cu") (net 1))
   (segment (start 71.944 95.758) (end 60.452 95.758) (width 1.016) (layer "F.Cu") (net 1))
   (segment (start 84.901989 28.513989) (end 85.622486 27.793518) (width 0.3048) (layer "F.Cu") (net 1))
-  (segment (start 83.693 38.564922) (end 82.212078 37.084) (width 0.3048) (layer "F.Cu") (net 1))
   (segment (start 78.328 134.716) (end 78.232 134.62) (width 0.25) (layer "F.Cu") (net 1))
   (segment (start 60.452 95.758) (end 59.436 94.742) (width 1.016) (layer "F.Cu") (net 1))
   (segment (start 84.901989 28.513989) (end 83.82 27.432) (width 0.3048) (layer "F.Cu") (net 1))
   (segment (start 113.284 32.004) (end 121.92 32.004) (width 1.016) (layer "F.Cu") (net 1))
-  (segment (start 84.287919 30.48) (end 84.901989 30.48) (width 0.3048) (layer "F.Cu") (net 1))
+  (segment (start 83.228078 38.1) (end 80.01 38.1) (width 0.3048) (layer "F.Cu") (net 1))
   (segment (start 73.66 71.628) (end 73.66 73.214) (width 1.016) (layer "F.Cu") (net 1))
-  (segment (start 80.772 37.084) (end 80.772 33.995919) (width 0.3048) (layer "F.Cu") (net 1))
   (segment (start 59.436 94.742) (end 59.436 91.948) (width 1.016) (layer "F.Cu") (net 1))
   (segment (start 78.232 143.398) (end 87.33 152.496) (width 1.016) (layer "F.Cu") (net 1))
   (segment (start 110.4235 32.004) (end 110.3575 32.07) (width 1.016) (layer "F.Cu") (net 1))
+  (segment (start 80.01 38.1) (end 79.502 37.592) (width 0.3048) (layer "F.Cu") (net 1))
   (segment (start 73.66 73.214) (end 73.725 73.279) (width 1.016) (layer "F.Cu") (net 1))
   (segment (start 78.39 99.156) (end 78.39 97.948) (width 1.016) (layer "F.Cu") (net 1))
   (segment (start 78.39 97.948) (end 74.803 94.361) (width 1.016) (layer "F.Cu") (net 1))
   (segment (start 78.232 134.62) (end 78.232 99.314) (width 1.016) (layer "F.Cu") (net 1))
+  (segment (start 83.693 38.564922) (end 83.228078 38.1) (width 0.3048) (layer "F.Cu") (net 1))
   (segment (start 78.232 134.62) (end 78.232 143.398) (width 1.016) (layer "F.Cu") (net 1))
+  (segment (start 84.287919 30.48) (end 84.901989 30.48) (width 0.3048) (layer "F.Cu") (net 1))
+  (segment (start 79.502 37.592) (end 79.502 35.265919) (width 0.3048) (layer "F.Cu") (net 1))
   (segment (start 87.33 116.936) (end 86.98 116.586) (width 1.016) (layer "F.Cu") (net 1))
   (segment (start 78.232 99.314) (end 78.39 99.156) (width 1.016) (layer "F.Cu") (net 1))
   (segment (start 86.98 116.586) (end 78.232 116.586) (width 1.016) (layer "F.Cu") (net 1))
   (segment (start 85.622486 27.793518) (end 85.622486 27.432) (width 0.3048) (layer "F.Cu") (net 1))
-  (segment (start 83.693 39.559001) (end 83.693 38.564922) (width 0.3048) (layer "F.Cu") (net 1))
   (segment (start 74.803 92.899) (end 71.944 95.758) (width 1.016) (layer "F.Cu") (net 1))
   (via (at 73.66 71.628) (size 0.6096) (drill 0.3048) (layers "F.Cu" "B.Cu") (net 1))
@@
   (segment (start 80.772 79.756) (end 86.868 73.66) (width 0.2032) (layer "B.Cu") (net 18))
   (segment (start 80.771989 79.756) (end 80.772 79.756) (width 0.2032) (layer "B.Cu") (net 18))
-  (segment (start 76.2 77.216) (end 77.343 78.359) (width 0.2032) (layer "F.Cu") (net 19))
+  (segment (start 76.2 69.85) (end 76.2 76.303347) (width 0.2032) (layer "F.Cu") (net 19))
   (segment (start 92.345 74.708) (end 90.456 74.708) (width 0.2032) (layer "F.Cu") (net 19))
-  (segment (start 77.343 78.359) (end 78.675 78.359) (width 0.2032) (layer "F.Cu") (net 19))
+  (segment (start 76.2 76.303347) (end 78.255653 78.359) (width 0.2032) (layer "F.Cu") (net 19))
   (segment (start 89.408 73.66) (end 89.408 72.136) (width 0.2032) (layer "F.Cu") (net 19))
+  (segment (start 78.255653 78.359) (end 78.675 78.359) (width 0.2032) (layer "F.Cu") (net 19))
   (segment (start 90.456 74.708) (end 89.408 73.66) (width 0.2032) (layer "F.Cu") (net 19))
   (segment (start 78.675 79.629) (end 78.675 78.359) (width 0.3048) (layer "F.Cu") (net 19))
-  (via (at 76.2 77.216) (size 0.6096) (drill 0.3048) (layers "F.Cu" "B.Cu") (net 19))
+  (via (at 76.2 69.85) (size 0.6096) (drill 0.3048) (layers "F.Cu" "B.Cu") (net 19))
   (via (at 89.408 72.136) (size 0.6096) (drill 0.3048) (layers "F.Cu" "B.Cu") (net 19))
   (segment (start 88.6391 72.9049) (end 89.408 72.136) (width 0.2032) (layer "B.Cu") (net 19))
-  (segment (start 76.2 77.216) (end 76.708 77.216) (width 0.2032) (layer "B.Cu") (net 19))
-  (segment (start 81.0191 72.9049) (end 88.6391 72.9049) (width 0.2032) (layer "B.Cu") (net 19))
-  (segment (start 76.708 77.216) (end 81.0191 72.9049) (width 0.2032) (layer "B.Cu") (net 19))
+  (segment (start 79.248 69.85) (end 82.3029 72.9049) (width 0.2032) (layer "B.Cu") (net 19))
+  (segment (start 82.3029 72.9049) (end 88.6391 72.9049) (width 0.2032) (layer "B.Cu") (net 19))
+  (segment (start 76.2 69.85) (end 79.248 69.85) (width 0.2032) (layer "B.Cu") (net 19))
   (segment (start 64.516 140.716) (end 89.329997 140.716) (width 1.016) (layer "B.Cu") (net 20))
   (segment (start 89.408 75.184) (end 89.732 75.508) (width 0.2032) (layer "F.Cu") (net 21))
@@
   (segment (start 89.617741 39.624) (end 88.392 39.624) (width 0.2032) (layer "B.Cu") (net 45))
   (segment (start 89.512871 65.128871) (end 89.512871 49.888871) (width 0.2032) (layer "B.Cu") (net 45))
+  (segment (start 82.423 34.925) (end 82.423 34.609) (width 0.2032) (layer "F.Cu") (net 46))
   (segment (start 93.72 72.13) (end 90.678 69.088) (width 0.2032) (layer "F.Cu") (net 46))
+  (segment (start 80.772 36.576) (end 82.423 34.925) (width 0.2032) (layer "F.Cu") (net 46))
   (segment (start 93.72 71.876) (end 93.72 72.533) (width 0.2032) (layer "F.Cu") (net 46))
-  (segment (start 82.423 35.179) (end 82.423 34.609) (width 0.2032) (layer "F.Cu") (net 46))
-  (segment (start 84.328 37.084) (end 82.423 35.179) (width 0.2032) (layer "F.Cu") (net 46))
   (segment (start 93.72 72.533) (end 93.72 72.13) (width 0.2032) (layer "F.Cu") (net 46))
-  (via (at 84.328 37.084) (size 0.6096) (drill 0.3048) (layers "F.Cu" "B.Cu") (net 46))
+  (via (at 80.772 36.576) (size 0.6096) (drill 0.3048) (layers "F.Cu" "B.Cu") (net 46))
   (via (at 90.678 69.088) (size 0.6096) (drill 0.3048) (layers "F.Cu" "B.Cu") (net 46))
-  (segment (start 80.772 39.624) (end 80.772 41.656) (width 0.2032) (layer "B.Cu") (net 46))
-  (segment (start 84.328 37.084) (end 83.312 37.084) (width 0.2032) (layer "B.Cu") (net 46))
-  (segment (start 83.312 37.084) (end 80.772 39.624) (width 0.2032) (layer "B.Cu") (net 46))
-  (segment (start 89.662 68.072) (end 88.9 68.072) (width 0.2032) (layer "B.Cu") (net 46))
+  (segment (start 90.932 47.752) (end 88.9 49.784) (width 0.2032) (layer "B.Cu") (net 46))
+  (segment (start 88.9 68.072) (end 89.662 68.072) (width 0.2032) (layer "B.Cu") (net 46))
+  (segment (start 80.772 36.576) (end 80.772 41.656) (width 0.2032) (layer "B.Cu") (net 46))
+  (segment (start 80.772 41.656) (end 90.932 41.656) (width 0.2032) (layer "B.Cu") (net 46))
+  (segment (start 88.9 49.784) (end 88.9 68.072) (width 0.2032) (layer "B.Cu") (net 46))
   (segment (start 90.932 41.656) (end 90.932 47.752) (width 0.2032) (layer "B.Cu") (net 46))
-  (segment (start 90.932 47.752) (end 88.9 49.784) (width 0.2032) (layer "B.Cu") (net 46))
-  (segment (start 80.772 41.656) (end 90.932 41.656) (width 0.2032) (layer "B.Cu") (net 46))
-  (segment (start 90.678 69.088) (end 89.662 68.072) (width 0.2032) (layer "B.Cu") (net 46))
-  (segment (start 88.9 49.784) (end 88.9 68.072) (width 0.2032) (layer "B.Cu") (net 46))
+  (segment (start 89.662 68.072) (end 90.678 69.088) (width 0.2032) (layer "B.Cu") (net 46))
   (segment (start 118.364 89.916) (end 121.412 86.868) (width 0.3048) (layer "F.Cu") (net 47))
   (segment (start 114.046 98.806) (end 117.348 95.504) (width 0.3048) (layer "F.Cu") (net 47))

Commit message: V6 Notas de silkscreen añadidas
Routing:
- net GND: track 89.1 -> 90.0 mm
Other:
- board text added: "- LEDBAR1"
- board text added: "- MTR 0.5A"
- board text added: "- MTR 1A"
- board text added: "12V"
- board text added: "5V"
- board text added: "6V"
- board text added: "BKGD"
- board text added: "COM"
- board text added: "D1"
- board text added: "D2"
- board text added: "D3"
- board text added: "GND"
- board text added: "GND1"
- board text added: "LDR_PIN1"
- board text added: "LDR_PIN2"
- board text added: "LVLHI"
- board text added: "LVLLO"
- board text added: "N.C"
- board text added: "N.O"
- board text added: "PH IN"
- board text added: "RST"
- board text added: "RX"
- board text added: "SCL"
- board text added: "SDA"
- board text added: "TDS IN"
- board text added: "TEMP & HUM"
- board text added: "TX"
