File: LIFFY/KiCAD/LIFFY_KICAD/LIFFY_KICAD.kicad_sch (KiCad schematic)
At the start: 13 parts, among them IC1 MC9S08MP16xLC, J1 VIN, J14 VIN2, J8 5V_OUT, Y1 Crystal 4 MHz

Commit message: V4.5 Fixed
Parts:
- removed R8: 10K, Resistor_SMD:R_0201_0603Metric, symbol Device:R
- removed RV4: Varistor_6V, Capacitor_SMD:C_0805_2012Metric, symbol Device:Varistor
- added L2: 27n, Inductor_SMD:L_0805_2012Metric, symbol Device:L
Connections:
- net +5V: now also L2.1; no longer C7.2, IC1.21 (VDDA/VREFH)
- net at C1.2, R7.2, Y1.2: now also IC1.27 (PTE5/XTAL)
- new net: C7.2, IC1.21 (VDDA/VREFH), L2.2
