File: LIFFY/KiCAD/LIFFY_KICAD/prog&com_pins.kicad_sch (KiCad schematic)
At the start: 9 parts, among them J15 Program_Pins, J16 CONN_I2C, J21 CONN_UART

Commit message: V4.5 Fixed
Parts:
- J15, J16, J21: footprint Connector_PinHeader_1.00mm:PinHeader_1x04_P1.00mm_Vertical -> Connector_PinHeader_2.54mm:PinHeader_1x04_P2.54mm_Vertical
Changed lines of the file:
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@@
     (property "Reference" "J16" (id 0) (at 94.615 121.92 0))
     (property "Value" "CONN_I2C" (id 1) (at 94.615 124.46 0))
-    (property "Footprint" "Connector_PinHeader_1.00mm:PinHeader_1x04_P1.00mm_Vertical" (id 2) (at 93.98 129.54 0)
+    (property "Footprint" "Connector_PinHeader_2.54mm:PinHeader_1x04_P2.54mm_Vertical" (id 2) (at 93.98 129.54 0)
       (effects (font (size 1.27 1.27)) hide)
     )
@@
     (property "Reference" "J21" (id 0) (at 147.955 88.9 0))
     (property "Value" "CONN_UART" (id 1) (at 147.955 91.44 0))
-    (property "Footprint" "Connector_PinHeader_1.00mm:PinHeader_1x04_P1.00mm_Vertical" (id 2) (at 147.32 96.52 0)
+    (property "Footprint" "Connector_PinHeader_2.54mm:PinHeader_1x04_P2.54mm_Vertical" (id 2) (at 147.32 96.52 0)
       (effects (font (size 1.27 1.27)) hide)
     )
@@
     (property "Reference" "J15" (id 0) (at 94.615 44.45 0))
     (property "Value" "Program_Pins" (id 1) (at 94.615 46.99 0))
-    (property "Footprint" "Connector_PinHeader_1.00mm:PinHeader_1x04_P1.00mm_Vertical" (id 2) (at 93.98 52.07 0)
+    (property "Footprint" "Connector_PinHeader_2.54mm:PinHeader_1x04_P2.54mm_Vertical" (id 2) (at 93.98 52.07 0)
       (effects (font (size 1.27 1.27)) hide)
     )

Commit message: V3 Fixed
Parts:
- J15, J16, J21: footprint Connector_PinHeader_2.54mm:PinHeader_1x04_P2.54mm_Vertical -> Connector_PinHeader_1.00mm:PinHeader_1x04_P1.00mm_Vertical
Changed lines of the file:
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@@
     (property "Reference" "J16" (id 0) (at 94.615 121.92 0))
     (property "Value" "CONN_I2C" (id 1) (at 94.615 124.46 0))
-    (property "Footprint" "Connector_PinHeader_2.54mm:PinHeader_1x04_P2.54mm_Vertical" (id 2) (at 93.98 129.54 0)
+    (property "Footprint" "Connector_PinHeader_1.00mm:PinHeader_1x04_P1.00mm_Vertical" (id 2) (at 93.98 129.54 0)
       (effects (font (size 1.27 1.27)) hide)
     )
@@
     (property "Reference" "J21" (id 0) (at 147.955 88.9 0))
     (property "Value" "CONN_UART" (id 1) (at 147.955 91.44 0))
-    (property "Footprint" "Connector_PinHeader_2.54mm:PinHeader_1x04_P2.54mm_Vertical" (id 2) (at 147.32 96.52 0)
+    (property "Footprint" "Connector_PinHeader_1.00mm:PinHeader_1x04_P1.00mm_Vertical" (id 2) (at 147.32 96.52 0)
       (effects (font (size 1.27 1.27)) hide)
     )
@@
     (property "Reference" "J15" (id 0) (at 94.615 44.45 0))
     (property "Value" "Program_Pins" (id 1) (at 94.615 46.99 0))
-    (property "Footprint" "Connector_PinHeader_2.54mm:PinHeader_1x04_P2.54mm_Vertical" (id 2) (at 93.98 52.07 0)
+    (property "Footprint" "Connector_PinHeader_1.00mm:PinHeader_1x04_P1.00mm_Vertical" (id 2) (at 93.98 52.07 0)
       (effects (font (size 1.27 1.27)) hide)
     )
